File: Numpad.sch (KiCad schematic (older format))
At the start: 44 parts, among them SW1 SW_Push, SW10 SW_Push, SW11 SW_Push, SW12 SW_Push, SW13 SW_Push, SW14 SW_Push, SW15 SW_Push, SW16 SW_Push, SW17 SW_Push, SW18 SW_Push, SW19 SW_Push, SW2 SW_Push, SW20 SW_Push, SW21 SW_Push, SW22 SW_Push, SW3 SW_Push, SW4 SW_Push, SW5 SW_Push, SW6 SW_Push, SW7 SW_Push, SW8 SW_Push, SW9 SW_Push, U1 ProMicro

Commit message: Switched to standalone STM32F103
Parts:
- removed SW1: SW_Push, Button_Switch_THT:SW_PUSH_6mm, symbol Switch:SW_Push
- removed U1: ProMicro, ProMicro:ProMicro, symbol ProMicro:ProMicro
- added C1, C10, C2, C3, C4, C6, C7: 100nf, symbol Device:C_Small
- added C11, C12, C5: 1uf, symbol Device:C_Small
- added C8, C9: C_Small, symbol Device:C_Small
- added F1: 500ma, symbol Device:Polyfuse_Small
- added H1, H2, H3, H4: MountingHole_Pad, symbol Mechanical:MountingHole_Pad
- added J1: SWD, symbol Connector:Conn_01x03_Male
- added J2: USB4085-GF-A_REVA, GCT_USB4085-GF-A_REVA, symbol USB4085:USB4085-GF-A_REVA
- added R1: 10k, symbol Device:R_Small_US
- added R2, R3: 5.1K, symbol Device:R_Small_US
- added R4, R5: 5, symbol Device:R_Small_US
- added U1: SRV05-4, Package_TO_SOT_SMD:SOT-23-6, symbol Power_Protection:SRV05-4
- added U2: STM32F103C8Tx, Package_QFP:LQFP-48_7x7mm_P0.5mm, symbol MCU_ST_STM32F1:STM32F103C8Tx
- added U3: XC6206PxxxMR, Package_TO_SOT_SMD:SOT-23, symbol Regulator_Linear:XC6206PxxxMR
- added Y1: 8MHz, symbol Device:Crystal_Small
- renumbered SW2 to SW1, SW11 to SW10, SW12 to SW11, SW13 to SW12, SW14 to SW13, SW15 to SW14, SW16 to SW15, SW17 to SW16, SW18 to SW17, SW19 to SW18, SW20 to SW19, SW3 to SW2, SW21 to SW20, SW22 to SW21, SW4 to SW3, SW5 to SW4, SW6 to SW5, SW7 to SW6, SW8 to SW7, SW9 to SW8, SW10 to SW9
Connections:
- net labels added: +3.3V, +5V, CC1, CC2, DA+, DA-, DB+, DB-, GND, VBAT, VDD1, VDD2, VDD3, VDDA
- wire segments 69 -> 124
- no-connect marks 11 -> 25
Other:
- note added: "SWDCLK"
- note added: "SWDIO\n"

Commit message: Assigned SMD components and generated netlist
Parts:
- C1, C10, C11, C12, C2, C3, C4, C5, C6, C7: footprint (none) -> Capacitor_SMD:C_0402_1005Metric
- C8, C9: value C_Small -> 20pf; footprint (none) -> Capacitor_SMD:C_0402_1005Metric
- D1, D10, D11, D12, D13, D14, D15, D16, D17, D18, D19, D2, D20, D21, D3, D4, D5, D6, D7, D8, D9: footprint Diode_THT:D_DO-35_SOD27_P7.62mm_Horizontal -> Diode_SMD:D_SOD-123
- F1: footprint (none) -> Fuse:Fuse_0805_2012Metric
- H1, H2, H3, H4: footprint (none) -> MountingHole:MountingHole_3.2mm_M3_Pad
- J1: footprint (none) -> Connector_PinHeader_1.27mm:PinHeader_1x03_P1.27mm_Horizontal
- J2: footprint GCT_USB4085-GF-A_REVA -> USB4085:GCT_USB4085-GF-A_REVA
- R1, R2, R3, R4, R5: footprint (none) -> Resistor_SMD:R_0402_1005Metric
- Y1: footprint (none) -> Crystal:Crystal_SMD_5032-2Pin_5.0x3.2mm

Commit message: Finished
Parts:
- removed F1: 500ma, Fuse:Fuse_0805_2012Metric, symbol Device:Polyfuse_Small
- removed R4, R5: 5, Resistor_SMD:R_0402_1005Metric, symbol Device:R_Small_US
Connections:
- net DB+ is gone; now on net DA+: U2.33 (PA12)
- net DB- is gone; now on net DA-: U2.32 (PA11)
- net +5V: now also J2.A4 (VBUS), J2.A9 (VBUS), J2.B4 (VBUS), J2.B9 (VBUS)
- net DA+: now also U1.4 (IO3); no longer U1.6 (IO4)
- net DA-: now also U1.6 (IO4); no longer U1.4 (IO3)
- net GND: now also J1.1 (Pin_1); no longer J1.3 (Pin_3)
- net at U2.34 (PA13): now also J1.3 (Pin_3); no longer J1.1 (Pin_1)
Other:
- moved on the sheet: R2, R3
Changed lines of the file:
@@
 $EndComp
 Connection ~ 7150 4900
-Text Label 6850 1900 1    50   ~ 0
-VBAT
-Text Label 6950 1900 1    50   ~ 0
-VDD1
-Text Label 7050 1900 1    50   ~ 0
-VDD2
-Text Label 7150 1900 1    50   ~ 0
-VDD3
-Text Label 7250 1900 1    50   ~ 0
-VDDA
-Text Label 1050 1400 3    50   ~ 0
-VBAT
-Text Label 1450 1400 3    50   ~ 0
-VDD1
-Text Label 1850 1400 3    50   ~ 0
-VDD2
-Text Label 2250 1400 3    50   ~ 0
-VDD3
-Text Label 2650 1400 3    50   ~ 0
-VDDA
 $Comp
 L Device:C_Small C1
@@
 F 3 "~" H 8200 4600 50  0001 C CNN
 	1    8200 4600
-	-1   0    0    -1
+	-1   0    0    1
 $EndComp
 Wire Wire Line
@@
 	1    0    0    -1
 $EndComp
-$Comp
-L Device:Polyfuse_Small F1
-U 1 1 5E41D6AD
-P 9200 3250
-F 0 "F1" V 8995 3250 50  0000 C CNN
-F 1 "500ma" V 9086 3250 50  0000 C CNN
-F 2 "Fuse:Fuse_0805_2012Metric" H 9250 3050 50  0001 L CNN
-F 3 "~" H 9200 3250 50  0001 C CNN
-	1    9200 3250
-	0    -1   1    0
-$EndComp
-Wire Wire Line
-	9300 3250 9350 3250
-Wire Wire Line
-	9100 3250 8850 3250
 Wire Wire Line
 	8850 3250 8850 3100
@@
 $EndComp
 $Comp
-L Device:R_Small_US R5
-U 1 1 5E43E41A
-P 9250 3950
-F 0 "R5" V 9045 3950 50  0000 C CNN
-F 1 "5" V 9136 3950 50  0000 C CNN
-F 2 "Resistor_SMD:R_0402_1005Metric" H 9250 3950 50  0001 C CNN
-F 3 "~" H 9250 3950 50  0001 C CNN
-	1    9250 3950
-	0    1    1    0
-$EndComp
-$Comp
-L Device:R_Small_US R4
-U 1 1 5E43FC67
-P 9250 3650
-F 0 "R4" V 9045 3650 50  0000 C CNN
-F 1 "5" V 9136 3650 50  0000 C CNN
-F 2 "Resistor_SMD:R_0402_1005Metric" H 9250 3650 50  0001 C CNN
-F 3 "~" H 9250 3650 50  0001 C CNN
-	1    9250 3650
-	0    1    1    0
-$EndComp
-$Comp
 L Device:R_Small_US R2
 U 1 1 5E4574F8
-P 8350 2250
-F 0 "R2" V 8145 2250 50  0000 C CNN
-F 1 "5.1K" V 8236 2250 50  0000 C CNN
-F 2 "Resistor_SMD:R_0402_1005Metric" H 8350 2250 50  0001 C CNN
-F 3 "~" H 8350 2250 50  0001 C CNN
-	1    8350 2250
+P 8450 3600
+F 0 "R2" V 8245 3600 50  0000 C CNN
+F 1 "5.1K" V 8336 3600 50  0000 C CNN
+F 2 "Resistor_SMD:R_0402_1005Metric" H 8450 3600 50  0001 C CNN
+F 3 "~" H 8450 3600 50  0001 C CNN
+	1    8450 3600
 	0    1    1    0
 $EndComp
@@
 L power:GND #PWR018
 U 1 1 5E484A5F
-P 8250 2400
-F 0 "#PWR018" H 8250 2150 50  0001 C CNN
-F 1 "GND" V 8255 2272 50  0000 R CNN
-F 2 "" H 8250 2400 50  0001 C CNN
-F 3 "" H 8250 2400 50  0001 C CNN
-	1    8250 2400
+P 8350 3750
+F 0 "#PWR018" H 8350 3500 50  0001 C CNN
+F 1 "GND" V 8355 3622 50  0000 R CNN
+F 2 "" H 8350 3750 50  0001 C CNN
+F 3 "" H 8350 3750 50  0001 C CNN
+	1    8350 3750
 	0    1    1    0
 $EndComp
@@
 	1    0    0    -1
 $EndComp
-$Comp
-L Power_Protection:SRV05-4 U1
-U 1 1 5E4C0D35
-P 4800 1550
-F 0 "U1" H 4800 2231 50  0000 C CNN
-F 1 "SRV05-4" H 4800 2140 50  0000 C CNN
-F 2 "Package_TO_SOT_SMD:SOT-23-6" H 5500 1100 50  0001 C CNN
-F 3 "http://www.onsemi.com/pub/Collateral/SRV05-4-D.PDF" H 4800 1550 50  0001 C CNN
-	1    4800 1550
-	1    0    0    -1
-$EndComp
 NoConn ~ 4300 1450
 NoConn ~ 4300 1650
@@
 	0    1    1    0
 $EndComp
-Text Label 5300 1450 0    50   ~ 0
-DA-
-Text Label 5300 1650 0    50   ~ 0
-DA+
 $Comp
 L power:GND #PWR014
@@
 	1    0    0    -1
 $EndComp
-Text Label 9450 3950 3    50   ~ 0
-DA-
-Text Label 9450 3650 3    50   ~ 0
-DA+
 Text GLabel 6350 4400 0    50   Input ~ 0
 col4
@@
 L Device:R_Small_US R3
 U 1 1 5E458E16
-P 8350 2550
-F 0 "R3" V 8555 2550 50  0000 C CNN
-F 1 "5.1K" V 8464 2550 50  0000 C CNN
-F 2 "Resistor_SMD:R_0402_1005Metric" H 8350 2550 50  0001 C CNN
-F 3 "~" H 8350 2550 50  0001 C CNN
-	1    8350 2550
+P 8450 3900
+F 0 "R3" V 8655 3900 50  0000 C CNN
+F 1 "5.1K" V 8564 3900 50  0000 C CNN
+F 2 "Resistor_SMD:R_0402_1005Metric" H 8450 3900 50  0001 C CNN
+F 3 "~" H 8450 3900 50  0001 C CNN
+	1    8450 3900
 	0    -1   -1   0
 $EndComp
@@
 	10200 850  10200 1050
 Wire Wire Line
-	8250 2250 8250 2400
-Wire Wire Line
-	8250 2400 8250 2550
-Connection ~ 8250 2400
-Text Label 8450 2250 0    50   ~ 0
+	8350 3600 8350 3750
+Wire Wire Line
+	8350 3750 8350 3900
+Connection ~ 8350 3750
+Text Label 8550 3600 0    50   ~ 0
 CC1
-Text Label 8450 2550 0    50   ~ 0
+Text Label 8550 3900 0    50   ~ 0
 CC2
 Text Label 9550 3450 2    50   ~ 0
@@
 Text Label 9550 3550 2    50   ~ 0
 CC2
-Wire Wire Line
-	9350 3650 9550 3650
 Connection ~ 9550 3650
-Wire Wire Line
-	9550 3950 9350 3950
 Connection ~ 9550 3950
-Wire Wire Line
-	9150 3650 9050 3650
-Wire Wire Line
-	9150 3950 9050 3950
-Text Label 9050 3650 2    50   ~ 0
-DB+
-Text Label 9050 3950 2    50   ~ 0
-DB-
-Text Label 7750 4300 0    50   ~ 0
-DB-
-Text Label 7750 4400 0    50   ~ 0
-DB+
 Wire Wire Line
 	7750 4300 7650 4300
@@
 	-1   0    0    1
 $EndComp
-Connection ~ 9350 3250
 Wire Wire Line
 	9350 3250 9550 3250
-$Comp
-L power:PWR_FLAG #FLG0103
-U 1 1 5E5E5740
-P 8850 3250
-F 0 "#FLG0103" H 8850 3325 50  0001 C CNN
-F 1 "PWR_FLAG" V 8850 3377 50  0000 L CNN
-F 2 "" H 8850 3250 50  0001 C CNN
-F 3 "~" H 8850 3250 50  0001 C CNN
-	1    8850 3250
-	0    -1   -1   0
-$EndComp
-Connection ~ 8850 3250
 Wire Wire Line
 	6350 2450 6000 2450
@@
 	0    -1   -1   0
 $EndComp
+Text GLabel 6850 1900 1    50   Input ~ 0
+VBAT
+Text GLabel 6950 1900 1    50   Input ~ 0
+VDD1
+Text GLabel 7050 1900 1    50   Input ~ 0
+VDD2
+Text GLabel 7150 1900 1    50   Input ~ 0
+VDD3
+Text GLabel 7250 1900 1    50   Input ~ 0
+VDDA
+Text GLabel 1050 1400 3    50   Input ~ 0
+VBAT
+Text GLabel 1450 1400 3    50   Input ~ 0
+VDD1
+Text GLabel 1850 1400 3    50   Input ~ 0
+VDD2
+Text GLabel 2250 1400 3    50   Input ~ 0
+VDD3
+Text GLabel 2650 1400 3    50   Input ~ 0
+VDDA
+Text GLabel 5300 1450 2    50   Input ~ 0
+DA+
+Text GLabel 5300 1650 2    50   Input ~ 0
+DA-
+$Comp
+L Power_Protection:SRV05-4 U1
+U 1 1 5E4C0D35
+P 4800 1550
+F 0 "U1" H 4800 2231 50  0000 C CNN
+F 1 "SRV05-4" H 4800 2140 50  0000 C CNN
+F 2 "Package_TO_SOT_SMD:SOT-23-6" H 5500 1100 50  0001 C CNN
+F 3 "http://www.onsemi.com/pub/Collateral/SRV05-4-D.PDF" H 4800 1550 50  0001 C CNN
+	1    4800 1550
+	1    0    0    -1
+$EndComp
+Text GLabel 9450 3650 3    50   Input ~ 0
+DA+
+Text GLabel 9450 3950 3    50   Input ~ 0
+DA-
+Text GLabel 9250 3650 0    50   Input ~ 0
+DB+
+Text GLabel 9250 3950 0    50   Input ~ 0
+DB-
+Text GLabel 7750 4300 2    50   Input ~ 0
+DB-
+Text GLabel 7750 4400 2    50   Input ~ 0
+DB+
+Wire Wire Line
+	9250 3650 9550 3650
+Wire Wire Line
+	9250 3950 9550 3950
+Wire Wire Line
+	9350 3250 8850 3250
+Connection ~ 9350 3250
 $EndSCHEMATC

Commit message: ground plane
Connections:
- net row3: now also U2.20 (PB2); no longer U2.46 (PB9)
- net row4: now also U2.19 (PB1); no longer U2.45 (PB8)
- net row5: now also U2.18 (PB0); no longer U2.43 (PB7)
- net row6: now also U2.17 (PA7); no longer U2.42 (PB6)
Changed lines of the file:
@@
 Text GLabel 6350 4300 0    50   Input ~ 0
 row1
-Text GLabel 6350 4100 0    50   Input ~ 0
+Text GLabel 6350 3400 0    50   Input ~ 0
 row3
-Text GLabel 6350 4000 0    50   Input ~ 0
+Text GLabel 6350 3300 0    50   Input ~ 0
 row4
-Text GLabel 6350 3900 0    50   Input ~ 0
+Text GLabel 6350 3200 0    50   Input ~ 0
 row5
-Text GLabel 6350 3800 0    50   Input ~ 0
+Text GLabel 7650 3900 2    50   Input ~ 0
 row6
 Text GLabel 6350 4200 0    50   Input ~ 0
@@
 NoConn ~ 6350 3600
 NoConn ~ 6350 3500
-NoConn ~ 6350 3400
-NoConn ~ 6350 3300
-NoConn ~ 6350 3200
+NoConn ~ 6350 4000
+NoConn ~ 6350 3900
+NoConn ~ 6350 3800
 NoConn ~ 7650 3200
 NoConn ~ 7650 3300
@@
 NoConn ~ 7650 3700
 NoConn ~ 7650 3800
-NoConn ~ 7650 3900
+NoConn ~ 6350 4100
 NoConn ~ 7650 4000
 NoConn ~ 7650 4100

Commit message: D+ pullup and some other things
Parts:
- added R4: 1.5K, Resistor_SMD:R_0402_1005Metric, symbol Device:R_Small_US
Connections:
- net +3V3: now also R4.1
- net DA+: now also R4.2
Changed lines of the file:
@@
 Text GLabel 9450 3950 3    50   Input ~ 0
 DA-
-Text GLabel 9250 3650 0    50   Input ~ 0
+Text GLabel 8950 3650 0    50   Input ~ 0
 DB+
-Text GLabel 9250 3950 0    50   Input ~ 0
+Text GLabel 8950 3950 0    50   Input ~ 0
 DB-
 Text GLabel 7750 4300 2    50   Input ~ 0
@@
 DB+
 Wire Wire Line
-	9250 3650 9550 3650
-Wire Wire Line
-	9250 3950 9550 3950
-Wire Wire Line
 	9350 3250 8850 3250
 Connection ~ 9350 3250
+Wire Wire Line
+	8950 3650 9300 3650
+Wire Wire Line
+	8950 3950 9550 3950
+$Comp
+L Device:R_Small_US R4
+U 1 1 5E36917C
+P 9100 3800
+F 0 "R4" V 9305 3800 50  0000 C CNN
+F 1 "1.5K" V 9214 3800 50  0000 C CNN
+F 2 "Resistor_SMD:R_0402_1005Metric" H 9100 3800 50  0001 C CNN
+F 3 "~" H 9100 3800 50  0001 C CNN
+	1    9100 3800
+	0    -1   -1   0
+$EndComp
+Wire Wire Line
+	9200 3800 9300 3800
+Wire Wire Line
+	9300 3800 9300 3650
+Connection ~ 9300 3650
+Wire Wire Line
+	9300 3650 9550 3650
+Wire Wire Line
+	9000 3800 8950 3800
+$Comp
+L power:+3.3V #PWR0101
+U 1 1 5E37570D
+P 8950 3800
+F 0 "#PWR0101" H 8950 3650 50  0001 C CNN
+F 1 "+3.3V" V 8965 3928 50  0000 L CNN
+F 2 "" H 8950 3800 50  0001 C CNN
+F 3 "" H 8950 3800 50  0001 C CNN
+	1    8950 3800
+	0    -1   -1   0
+$EndComp
 $EndSCHEMATC

Commit message: finalized v0.2
Parts:
- C1, C10, C2, C3, C4, C6, C7: LCSC (none) -> C1525
- C11, C12, C5: LCSC (none) -> C52923
- C8, C9: LCSC (none) -> C1554
- D1, D10, D11, D12, D13, D14, D15, D16, D17, D18, D19, D2, D20, D21, D3, D4, D5, D6, D7, D8, D9: LCSC (none) -> C81598
- R1: LCSC (none) -> C25744
- R2, R3: LCSC (none) -> C25905
- R4: LCSC (none) -> C25867
- U1: LCSC (none) -> C85364
- U2: LCSC (none) -> C8734
- U3: LCSC (none) -> C5446
- Y1: LCSC (none) -> C115962
Changed lines of the file:
@@
 F 2 "Diode_SMD:D_SOD-123" H 1650 5525 50  0001 C CNN
 F 3 "https://assets.nexperia.com/documents/data-sheet/1N4148_1N4448.pdf" H 1650 5700 50  0001 C CNN
+F 4 "C81598" H 1650 5700 50  0001 C CNN "LCSC"
 	1    1650 5700
 	1    0    0    -1
@@
 F 2 "Diode_SMD:D_SOD-123" H 1650 6175 50  0001 C CNN
 F 3 "https://assets.nexperia.com/documents/data-sheet/1N4148_1N4448.pdf" H 1650 6350 50  0001 C CNN
+F 4 "C81598" H 1650 6350 50  0001 C CNN "LCSC"
 	1    1650 6350
 	1    0    0    -1
@@
 F 2 "Diode_SMD:D_SOD-123" H 2450 4125 50  0001 C CNN
 F 3 "https://assets.nexperia.com/documents/data-sheet/1N4148_1N4448.pdf" H 2450 4300 50  0001 C CNN
+F 4 "C81598" H 2450 4300 50  0001 C CNN "LCSC"
 	1    2450 4300
 	1    0    0    -1
@@
 F 2 "Diode_SMD:D_SOD-123" H 2450 4825 50  0001 C CNN
 F 3 "https://assets.nexperia.com/documents/data-sheet/1N4148_1N4448.pdf" H 2450 5000 50  0001 C CNN
+F 4 "C81598" H 2450 5000 50  0001 C CNN "LCSC"
 	1    2450 5000
 	1    0    0    -1
@@
 F 2 "Diode_SMD:D_SOD-123" H 2450 5525 50  0001 C CNN
 F 3 "https://assets.nexperia.com/documents/data-sheet/1N4148_1N4448.pdf" H 2450 5700 50  0001 C CNN
+F 4 "C81598" H 2450 5700 50  0001 C CNN "LCSC"
 	1    2450 5700
 	1    0    0    -1
@@
 F 2 "Diode_SMD:D_SOD-123" H 2450 6175 50  0001 C CNN
 F 3 "https://assets.nexperia.com/documents/data-sheet/1N4148_1N4448.pdf" H 2450 6350 50  0001 C CNN
+F 4 "C81598" H 2450 6350 50  0001 C CNN "LCSC"
 	1    2450 6350
 	1    0    0    -1
@@
 F 2 "Diode_SMD:D_SOD-123" H 3200 4125 50  0001 C CNN
 F 3 "https://assets.nexperia.com/documents/data-sheet/1N4148_1N4448.pdf" H 3200 4300 50  0001 C CNN
+F 4 "C81598" H 3200 4300 50  0001 C CNN "LCSC"
 	1    3200 4300
 	1    0    0    -1
@@
 F 2 "Diode_SMD:D_SOD-123" H 3200 4825 50  0001 C CNN
 F 3 "https://assets.nexperia.com/documents/data-sheet/1N4148_1N4448.pdf" H 3200 5000 50  0001 C CNN
+F 4 "C81598" H 3200 5000 50  0001 C CNN "LCSC"
 	1    3200 5000
 	1    0    0    -1
@@
 F 2 "Diode_SMD:D_SOD-123" H 3200 5525 50  0001 C CNN
 F 3 "https://assets.nexperia.com/documents/data-sheet/1N4148_1N4448.pdf" H 3200 5700 50  0001 C CNN
+F 4 "C81598" H 3200 5700 50  0001 C CNN "LCSC"
 	1    3200 5700
 	1    0    0    -1
@@
 F 2 "Diode_SMD:D_SOD-123" H 3200 6175 50  0001 C CNN
 F 3 "https://assets.nexperia.com/documents/data-sheet/1N4148_1N4448.pdf" H 3200 6350 50  0001 C CNN
+F 4 "C81598" H 3200 6350 50  0001 C CNN "LCSC"
 	1    3200 6350
 	1    0    0    -1
@@
 F 2 "Diode_SMD:D_SOD-123" H 3200 6875 50  0001 C CNN
 F 3 "https://assets.nexperia.com/documents/data-sheet/1N4148_1N4448.pdf" H 3200 7050 50  0001 C CNN
+F 4 "C81598" H 3200 7050 50  0001 C CNN "LCSC"
 	1    3200 7050
 	1    0    0    -1
@@
 F 2 "Diode_SMD:D_SOD-123" H 4000 4125 50  0001 C CNN
 F 3 "https://assets.nexperia.com/documents/data-sheet/1N4148_1N4448.pdf" H 4000 4300 50  0001 C CNN
+F 4 "C81598" H 4000 4300 50  0001 C CNN "LCSC"
 	1    4000 4300
 	1    0    0    -1
@@
 F 2 "Diode_SMD:D_SOD-123" H 4000 4825 50  0001 C CNN
 F 3 "https://assets.nexperia.com/documents/data-sheet/1N4148_1N4448.pdf" H 4000 5000 50  0001 C CNN
+F 4 "C81598" H 4000 5000 50  0001 C CNN "LCSC"
 	1    4000 5000
 	1    0    0    -1
@@
 F 2 "Diode_SMD:D_SOD-123" H 4000 6175 50  0001 C CNN
 F 3 "https://assets.nexperia.com/documents/data-sheet/1N4148_1N4448.pdf" H 4000 6350 50  0001 C CNN
+F 4 "C81598" H 4000 6350 50  0001 C CNN "LCSC"
 	1    4000 6350
 	1    0    0    -1
@@
 F 2 "Diode_SMD:D_SOD-123" H 4000 3475 50  0001 C CNN
 F 3 "https://assets.nexperia.com/documents/data-sheet/1N4148_1N4448.pdf" H 4000 3650 50  0001 C CNN
+F 4 "C81598" H 4000 3650 50  0001 C CNN "LCSC"
 	1    4000 3650
 	1    0    0    -1
@@
 F 2 "Diode_SMD:D_SOD-123" H 3200 3475 50  0001 C CNN
 F 3 "https://assets.nexperia.com/documents/data-sheet/1N4148_1N4448.pdf" H 3200 3650 50  0001 C CNN
+F 4 "C81598" H 3200 3650 50  0001 C CNN "LCSC"
 	1    3200 3650
 	1    0    0    -1
@@
 F 2 "Diode_SMD:D_SOD-123" H 2450 3475 50  0001 C CNN
 F 3 "https://assets.nexperia.com/documents/data-sheet/1N4148_1N4448.pdf" H 2450 3650 50  0001 C CNN
+F 4 "C81598" H 2450 3650 50  0001 C CNN "LCSC"
 	1    2450 3650
 	1    0    0    -1
@@
 F 2 "Diode_SMD:D_SOD-123" H 1650 3475 50  0001 C CNN
 F 3 "https://assets.nexperia.com/documents/data-sheet/1N4148_1N4448.pdf" H 1650 3650 50  0001 C CNN
+F 4 "C81598" H 1650 3650 50  0001 C CNN "LCSC"
 	1    1650 3650
 	1    0    0    -1
@@
 F 2 "Diode_SMD:D_SOD-123" H 1650 4125 50  0001 C CNN
 F 3 "https://assets.nexperia.com/documents/data-sheet/1N4148_1N4448.pdf" H 1650 4300 50  0001 C CNN
+F 4 "C81598" H 1650 4300 50  0001 C CNN "LCSC"
 	1    1650 4300
 	1    0    0    -1
@@
 F 2 "Diode_SMD:D_SOD-123" H 1650 4825 50  0001 C CNN
 F 3 "https://assets.nexperia.com/documents/data-sheet/1N4148_1N4448.pdf" H 1650 5000 50  0001 C CNN
+F 4 "C81598" H 1650 5000 50  0001 C CNN "LCSC"
 	1    1650 5000
 	1    0    0    -1
@@
 F 2 "Diode_SMD:D_SOD-123" H 1650 6875 50  0001 C CNN
 F 3 "https://assets.nexperia.com/documents/data-sheet/1N4148_1N4448.pdf" H 1650 7050 50  0001 C CNN
+F 4 "C81598" H 1650 7050 50  0001 C CNN "LCSC"
 	1    1650 7050
 	1    0    0    -1
@@
 F 2 "Capacitor_SMD:C_0402_1005Metric" H 5900 2450 50  0001 C CNN
 F 3 "~" H 5900 2450 50  0001 C CNN
+F 4 "C1554" H 5900 2450 50  0001 C CNN "LCSC"
 	1    5900 2450
 	0    1    1    0
@@
 F 2 "Capacitor_SMD:C_0402_1005Metric" H 6350 1900 50  0001 C CNN
 F 3 "~" H 6350 1900 50  0001 C CNN
+F 4 "C1525" H 6350 1900 50  0001 C CNN "LCSC"
 	1    6350 1900
 	1    0    0    -1
@@
 F 2 "Resistor_SMD:R_0402_1005Metric" H 6250 2300 50  0001 C CNN
 F 3 "~" H 6250 2300 50  0001 C CNN
+F 4 "C25744" H 6250 2300 50  0001 C CNN "LCSC"
 	1    6250 2300
 	0    1    1    0
@@
 F 2 "Capacitor_SMD:C_0402_1005Metric" H 5900 2650 50  0001 C CNN
 F 3 "~" H 5900 2650 50  0001 C CNN
+F 4 "C1554" H 5900 2650 50  0001 C CNN "LCSC"
 	1    5900 2650
 	0    1    1    0
@@
 F 2 "Package_QFP:LQFP-48_7x7mm_P0.5mm" H 6450 2000 50  0001 R CNN
 F 3 "http://www.st.com/st-web-ui/static/active/en/resource/technical/document/datasheet/CD00161566.pdf" H 7050 3400 50  0001 C CNN
+F 4 "C8734" H 7050 3400 50  0001 C CNN "LCSC"
 	1    7050 3400
 	1    0    0    -1
@@
 F 2 "Capacitor_SMD:C_0402_1005Metric" H 1150 1300 50  0001 C CNN
 F 3 "~" H 1150 1300 50  0001 C CNN
+F 4 "C1525" H 1150 1300 50  0001 C CNN "LCSC"
 	1    1150 1300
 	0    1    1    0
@@
 F 2 "Capacitor_SMD:C_0402_1005Metric" H 1550 1300 50  0001 C CNN
 F 3 "~" H 1550 1300 50  0001 C CNN
+F 4 "C1525" H 1550 1300 50  0001 C CNN "LCSC"
 	1    1550 1300
 	0    1    1    0
@@
 F 2 "Capacitor_SMD:C_0402_1005Metric" H 1950 1300 50  0001 C CNN
 F 3 "~" H 1950 1300 50  0001 C CNN
+F 4 "C1525" H 1950 1300 50  0001 C CNN "LCSC"
 	1    1950 1300
 	0    1    1    0
@@
 F 2 "Capacitor_SMD:C_0402_1005Metric" H 2350 1300 50  0001 C CNN
 F 3 "~" H 2350 1300 50  0001 C CNN
+F 4 "C1525" H 2350 1300 50  0001 C CNN "LCSC"
 	1    2350 1300
 	0    1    1    0
@@
 F 2 "Capacitor_SMD:C_0402_1005Metric" H 2750 1300 50  0001 C CNN
 F 3 "~" H 2750 1300 50  0001 C CNN
+F 4 "C1525" H 2750 1300 50  0001 C CNN "LCSC"
 	1    2750 1300
 	0    1    1    0
@@
 F 2 "Capacitor_SMD:C_0402_1005Metric" H 3200 1300 50  0001 C CNN
 F 3 "~" H 3200 1300 50  0001 C CNN
+F 4 "C1525" H 3200 1300 50  0001 C CNN "LCSC"
 	1    3200 1300
 	0    1    1    0
@@
 F 2 "Capacitor_SMD:C_0402_1005Metric" H 2750 1000 50  0001 C CNN
 F 3 "~" H 2750 1000 50  0001 C CNN
+F 4 "C52923" H 2750 1000 50  0001 C CNN "LCSC"
 	1    2750 1000
 	0    1    1    0
@@
 F 2 "Resistor_SMD:R_0402_1005Metric" H 8450 3600 50  0001 C CNN
 F 3 "~" H 8450 3600 50  0001 C CNN
+F 4 "C25905" H 8450 3600 50  0001 C CNN "LCSC"
 	1    8450 3600
 	0    1    1    0
@@
 F 2 "Package_TO_SOT_SMD:SOT-23" H 9100 1675 50  0001 C CIN
 F 3 "https://www.torexsemi.com/file/xc6206/XC6206.pdf" H 9100 1450 50  0001 C CNN
+F 4 "C5446" H 9100 1450 50  0001 C CNN "LCSC"
 	1    9100 1450
 	1    0    0    -1
@@
 F 2 "Capacitor_SMD:C_0402_1005Metric" H 8700 1600 50  0001 C CNN
 F 3 "~" H 8700 1600 50  0001 C CNN
+F 4 "C52923" H 8700 1600 50  0001 C CNN "LCSC"
 	1    8700 1600
 	1    0    0    1
@@
 F 2 "Capacitor_SMD:C_0402_1005Metric" H 9500 1600 50  0001 C CNN
 F 3 "~" H 9500 1600 50  0001 C CNN
+F 4 "C52923" H 9500 1600 50  0001 C CNN "LCSC"
 	1    9500 1600
 	1    0    0    -1
@@
 F 2 "Resistor_SMD:R_0402_1005Metric" H 8450 3900 50  0001 C CNN
 F 3 "~" H 8450 3900 50  0001 C CNN
+F 4 "C25905" H 8450 3900 50  0001 C CNN "LCSC"
 	1    8450 3900
 	0    -1   -1   0
@@
 F 2 "Crystal:Crystal_SMD_5032-2Pin_5.0x3.2mm" H 6000 2550 50  0001 C CNN
 F 3 "~" H 6000 2550 50  0001 C CNN
+F 4 "C115962" H 6000 2550 50  0001 C CNN "LCSC"
 	1    6000 2550
 	0    -1   -1   0
@@
 F 2 "Package_TO_SOT_SMD:SOT-23-6" H 5500 1100 50  0001 C CNN
 F 3 "http://www.onsemi.com/pub/Collateral/SRV05-4-D.PDF" H 4800 1550 50  0001 C CNN
+F 4 "C85364" H 4800 1550 50  0001 C CNN "LCSC"
 	1    4800 1550
 	1    0    0    -1
@@
 F 2 "Resistor_SMD:R_0402_1005Metric" H 9100 3800 50  0001 C CNN
 F 3 "~" H 9100 3800 50  0001 C CNN
+F 4 "C25867" H 9100 3800 50  0001 C CNN "LCSC"
 	1    9100 3800
 	0    -1   -1   0
