File: Numpad.sch (KiCad schematic (older format))
At the start: 68 parts, among them J1 SWD, J2 USB_C_Receptacle_USB2.0, U1 SRV05-4, U2 STM32F103C8Tx, U3 XC6206PxxxMR, Y1 8MHz

Commit message: Widened power traces, fixed some routing
Connections:
- net labels added: BOOT0, NRST, PD0, PD1, SWDCLK, SWDIO
- wire segments 123 -> 112
Other:
- note removed: "SWDCLK"
- note removed: "SWDIO\n"
- moved on the sheet: C10, C8, C9, R1, U2, Y1

Commit message: Annotated and reformatted schematic
Other:
- note added: "CC Pull-down"
- note added: "Data Lines"
- note added: "Debug Port"
- note added: "Decoupling Capacitors"
- note added: "ESD Protection"
- note added: "Key Matrix"
- note added: "MCU"
- note added: "Oscillator"
- note added: "Power Regulator"
- note added: "Support Circuitry"
- note added: "USB Port"
- moved on the sheet: C1, C10, C11, C12, C2, C3, C4, C5, C6, C7, C8, C9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

Commit message: Updated position of ESD protection diodes
Connections:
- no-connect marks 20 -> 18
Changed lines of the file:
@@
 	1    0    0    -1
 $EndComp
-NoConn ~ 5050 1700
-NoConn ~ 5050 1900
 $Comp
 L power:+5V #PWR013
@@
 Text GLabel 2850 2000 3    50   Input ~ 0
 VDDA
+Text GLabel 5050 1900 0    50   Input ~ 0
+DA+
 Text GLabel 6050 1700 2    50   Input ~ 0
-DA+
-Text GLabel 6050 1900 2    50   Input ~ 0
 DA-
 $Comp

Commit message: Changed LEDs to SOD323
Parts:
- D_0, D_1, D_2, D_3, D_4, D_5, D_6, D_7, D_8, D_9, D_BKSP1, D_DOT1, D_ENTER1, D_ESC1, D_FN1, D_MINUS1, D_NUMLK1, D_PLUS1, D_SLASH1, D_STAR1, D_TAB1: footprint Diode_SMD:D_SOD-123 -> Diode_SMD:D_SOD-323F
Changed lines of the file:
@@
 F 0 "D_4" H 1700 6366 50  0000 C CNN
 F 1 "1N4148" H 1700 6275 50  0000 C CNN
-F 2 "Diode_SMD:D_SOD-123" H 1700 5975 50  0001 C CNN
+F 2 "Diode_SMD:D_SOD-323F" H 1700 5975 50  0001 C CNN
 F 3 "https://assets.nexperia.com/documents/data-sheet/1N4148_1N4448.pdf" H 1700 6150 50  0001 C CNN
 F 4 "C81598" H 1700 6150 50  0001 C CNN "LCSC"
@@
 F 0 "D_1" H 1700 7016 50  0000 C CNN
 F 1 "1N4148" H 1700 6925 50  0000 C CNN
-F 2 "Diode_SMD:D_SOD-123" H 1700 6625 50  0001 C CNN
+F 2 "Diode_SMD:D_SOD-323F" H 1700 6625 50  0001 C CNN
 F 3 "https://assets.nexperia.com/documents/data-sheet/1N4148_1N4448.pdf" H 1700 6800 50  0001 C CNN
 F 4 "C81598" H 1700 6800 50  0001 C CNN "LCSC"
@@
 F 0 "D_SLASH1" H 2500 4966 50  0000 C CNN
 F 1 "1N4148" H 2500 4875 50  0000 C CNN
-F 2 "Diode_SMD:D_SOD-123" H 2500 4575 50  0001 C CNN
+F 2 "Diode_SMD:D_SOD-323F" H 2500 4575 50  0001 C CNN
 F 3 "https://assets.nexperia.com/documents/data-sheet/1N4148_1N4448.pdf" H 2500 4750 50  0001 C CNN
 F 4 "C81598" H 2500 4750 50  0001 C CNN "LCSC"
@@
 F 0 "D_8" H 2500 5666 50  0000 C CNN
 F 1 "1N4148" H 2500 5575 50  0000 C CNN
-F 2 "Diode_SMD:D_SOD-123" H 2500 5275 50  0001 C CNN
+F 2 "Diode_SMD:D_SOD-323F" H 2500 5275 50  0001 C CNN
 F 3 "https://assets.nexperia.com/documents/data-sheet/1N4148_1N4448.pdf" H 2500 5450 50  0001 C CNN
 F 4 "C81598" H 2500 5450 50  0001 C CNN "LCSC"
@@
 F 0 "D_5" H 2500 6366 50  0000 C CNN
 F 1 "1N4148" H 2500 6275 50  0000 C CNN
-F 2 "Diode_SMD:D_SOD-123" H 2500 5975 50  0001 C CNN
+F 2 "Diode_SMD:D_SOD-323F" H 2500 5975 50  0001 C CNN
 F 3 "https://assets.nexperia.com/documents/data-sheet/1N4148_1N4448.pdf" H 2500 6150 50  0001 C CNN
 F 4 "C81598" H 2500 6150 50  0001 C CNN "LCSC"
@@
 F 0 "D_2" H 2500 7016 50  0000 C CNN
 F 1 "1N4148" H 2500 6925 50  0000 C CNN
-F 2 "Diode_SMD:D_SOD-123" H 2500 6625 50  0001 C CNN
+F 2 "Diode_SMD:D_SOD-323F" H 2500 6625 50  0001 C CNN
 F 3 "https://assets.nexperia.com/documents/data-sheet/1N4148_1N4448.pdf" H 2500 6800 50  0001 C CNN
 F 4 "C81598" H 2500 6800 50  0001 C CNN "LCSC"
@@
 F 0 "D_STAR1" H 3300 4966 50  0000 C CNN
 F 1 "1N4148" H 3300 4875 50  0000 C CNN
-F 2 "Diode_SMD:D_SOD-123" H 3300 4575 50  0001 C CNN
+F 2 "Diode_SMD:D_SOD-323F" H 3300 4575 50  0001 C CNN
 F 3 "https://assets.nexperia.com/documents/data-sheet/1N4148_1N4448.pdf" H 3300 4750 50  0001 C CNN
 F 4 "C81598" H 3300 4750 50  0001 C CNN "LCSC"
@@
 F 0 "D_9" H 3300 5666 50  0000 C CNN
 F 1 "1N4148" H 3300 5575 50  0000 C CNN
-F 2 "Diode_SMD:D_SOD-123" H 3300 5275 50  0001 C CNN
+F 2 "Diode_SMD:D_SOD-323F" H 3300 5275 50  0001 C CNN
 F 3 "https://assets.nexperia.com/documents/data-sheet/1N4148_1N4448.pdf" H 3300 5450 50  0001 C CNN
 F 4 "C81598" H 3300 5450 50  0001 C CNN "LCSC"
@@
 F 0 "D_6" H 3300 6366 50  0000 C CNN
 F 1 "1N4148" H 3300 6275 50  0000 C CNN
-F 2 "Diode_SMD:D_SOD-123" H 3300 5975 50  0001 C CNN
+F 2 "Diode_SMD:D_SOD-323F" H 3300 5975 50  0001 C CNN
 F 3 "https://assets.nexperia.com/documents/data-sheet/1N4148_1N4448.pdf" H 3300 6150 50  0001 C CNN
 F 4 "C81598" H 3300 6150 50  0001 C CNN "LCSC"
@@
 F 0 "D_3" H 3300 7016 50  0000 C CNN
 F 1 "1N4148" H 3300 6925 50  0000 C CNN
-F 2 "Diode_SMD:D_SOD-123" H 3300 6625 50  0001 C CNN
+F 2 "Diode_SMD:D_SOD-323F" H 3300 6625 50  0001 C CNN
 F 3 "https://assets.nexperia.com/documents/data-sheet/1N4148_1N4448.pdf" H 3300 6800 50  0001 C CNN
 F 4 "C81598" H 3300 6800 50  0001 C CNN "LCSC"
@@
 F 0 "D_DOT1" H 3300 7716 50  0000 C CNN
 F 1 "1N4148" H 3300 7625 50  0000 C CNN
-F 2 "Diode_SMD:D_SOD-123" H 3300 7325 50  0001 C CNN
+F 2 "Diode_SMD:D_SOD-323F" H 3300 7325 50  0001 C CNN
 F 3 "https://assets.nexperia.com/documents/data-sheet/1N4148_1N4448.pdf" H 3300 7500 50  0001 C CNN
 F 4 "C81598" H 3300 7500 50  0001 C CNN "LCSC"
@@
 F 0 "D_MINUS1" H 4100 4966 50  0000 C CNN
 F 1 "1N4148" H 4100 4875 50  0000 C CNN
-F 2 "Diode_SMD:D_SOD-123" H 4100 4575 50  0001 C CNN
+F 2 "Diode_SMD:D_SOD-323F" H 4100 4575 50  0001 C CNN
 F 3 "https://assets.nexperia.com/documents/data-sheet/1N4148_1N4448.pdf" H 4100 4750 50  0001 C CNN
 F 4 "C81598" H 4100 4750 50  0001 C CNN "LCSC"
@@
 F 0 "D_PLUS1" H 4100 5666 50  0000 C CNN
 F 1 "1N4148" H 4100 5575 50  0000 C CNN
-F 2 "Diode_SMD:D_SOD-123" H 4100 5275 50  0001 C CNN
+F 2 "Diode_SMD:D_SOD-323F" H 4100 5275 50  0001 C CNN
 F 3 "https://assets.nexperia.com/documents/data-sheet/1N4148_1N4448.pdf" H 4100 5450 50  0001 C CNN
 F 4 "C81598" H 4100 5450 50  0001 C CNN "LCSC"
@@
 F 0 "D_ENTER1" H 4100 7016 50  0000 C CNN
 F 1 "1N4148" H 4100 6925 50  0000 C CNN
-F 2 "Diode_SMD:D_SOD-123" H 4100 6625 50  0001 C CNN
+F 2 "Diode_SMD:D_SOD-323F" H 4100 6625 50  0001 C CNN
 F 3 "https://assets.nexperia.com/documents/data-sheet/1N4148_1N4448.pdf" H 4100 6800 50  0001 C CNN
 F 4 "C81598" H 4100 6800 50  0001 C CNN "LCSC"
@@
 F 0 "D_BKSP1" H 4100 4316 50  0000 C CNN
 F 1 "1N4148" H 4100 4225 50  0000 C CNN
-F 2 "Diode_SMD:D_SOD-123" H 4100 3925 50  0001 C CNN
+F 2 "Diode_SMD:D_SOD-323F" H 4100 3925 50  0001 C CNN
 F 3 "https://assets.nexperia.com/documents/data-sheet/1N4148_1N4448.pdf" H 4100 4100 50  0001 C CNN
 F 4 "C81598" H 4100 4100 50  0001 C CNN "LCSC"
@@
 F 0 "D_TAB1" H 2500 4316 50  0000 C CNN
 F 1 "1N4148" H 2500 4225 50  0000 C CNN
-F 2 "Diode_SMD:D_SOD-123" H 2500 3925 50  0001 C CNN
+F 2 "Diode_SMD:D_SOD-323F" H 2500 3925 50  0001 C CNN
 F 3 "https://assets.nexperia.com/documents/data-sheet/1N4148_1N4448.pdf" H 2500 4100 50  0001 C CNN
 F 4 "C81598" H 2500 4100 50  0001 C CNN "LCSC"
@@
 F 0 "D_ESC1" H 1700 4316 50  0000 C CNN
 F 1 "1N4148" H 1700 4225 50  0000 C CNN
-F 2 "Diode_SMD:D_SOD-123" H 1700 3925 50  0001 C CNN
+F 2 "Diode_SMD:D_SOD-323F" H 1700 3925 50  0001 C CNN
 F 3 "https://assets.nexperia.com/documents/data-sheet/1N4148_1N4448.pdf" H 1700 4100 50  0001 C CNN
 F 4 "C81598" H 1700 4100 50  0001 C CNN "LCSC"
@@
 F 0 "D_NUMLK1" H 1700 4966 50  0000 C CNN
 F 1 "1N4148" H 1700 4875 50  0000 C CNN
-F 2 "Diode_SMD:D_SOD-123" H 1700 4575 50  0001 C CNN
+F 2 "Diode_SMD:D_SOD-323F" H 1700 4575 50  0001 C CNN
 F 3 "https://assets.nexperia.com/documents/data-sheet/1N4148_1N4448.pdf" H 1700 4750 50  0001 C CNN
 F 4 "C81598" H 1700 4750 50  0001 C CNN "LCSC"
@@
 F 0 "D_7" H 1700 5666 50  0000 C CNN
 F 1 "1N4148" H 1700 5575 50  0000 C CNN
-F 2 "Diode_SMD:D_SOD-123" H 1700 5275 50  0001 C CNN
+F 2 "Diode_SMD:D_SOD-323F" H 1700 5275 50  0001 C CNN
 F 3 "https://assets.nexperia.com/documents/data-sheet/1N4148_1N4448.pdf" H 1700 5450 50  0001 C CNN
 F 4 "C81598" H 1700 5450 50  0001 C CNN "LCSC"
@@
 Text GLabel 6250 5250 0    50   Input ~ 0
 row1
+Text GLabel 6250 5350 0    50   Input ~ 0
+row3
+Text GLabel 6250 4550 0    50   Input ~ 0
+row4
+Text GLabel 6250 4450 0    50   Input ~ 0
+row5
+Text GLabel 6250 4350 0    50   Input ~ 0
+row6
 Text GLabel 6250 5450 0    50   Input ~ 0
-row3
-Text GLabel 6250 4450 0    50   Input ~ 0
-row4
-Text GLabel 6250 4350 0    50   Input ~ 0
-row5
-Text GLabel 7550 5050 2    50   Input ~ 0
-row6
-Text GLabel 6250 5350 0    50   Input ~ 0
 row2
 NoConn ~ 6250 4850
@@
 F 0 "D_0" H 1700 7716 50  0000 C CNN
 F 1 "1N4148" H 1700 7625 50  0000 C CNN
-F 2 "Diode_SMD:D_SOD-123" H 1700 7325 50  0001 C CNN
+F 2 "Diode_SMD:D_SOD-323F" H 1700 7325 50  0001 C CNN
 F 3 "https://assets.nexperia.com/documents/data-sheet/1N4148_1N4448.pdf" H 1700 7500 50  0001 C CNN
 F 4 "C81598" H 1700 7500 50  0001 C CNN "LCSC"
@@
 F 0 "D_FN1" H 3300 4316 50  0000 C CNN
 F 1 "1N4148" H 3300 4225 50  0000 C CNN
-F 2 "Diode_SMD:D_SOD-123" H 3300 3925 50  0001 C CNN
+F 2 "Diode_SMD:D_SOD-323F" H 3300 3925 50  0001 C CNN
 F 3 "https://assets.nexperia.com/documents/data-sheet/1N4148_1N4448.pdf" H 3300 4100 50  0001 C CNN
 F 4 "C81598" H 3300 4100 50  0001 C CNN "LCSC"

Commit message: Fixed positioning of silkscreen labels
Parts:
- D_0, D_1, D_2, D_3, D_4, D_5, D_6, D_7, D_8, D_9, D_BKSP1, D_DOT1, D_ENTER1, D_ESC1, D_FN1, D_MINUS1, D_NUMLK1, D_PLUS1, D_SLASH1, D_STAR1, D_TAB1: LCSC C81598 -> C2128
Changed lines of the file:
@@
 F 2 "Diode_SMD:D_SOD-323F" H 1700 5975 50  0001 C CNN
 F 3 "https://assets.nexperia.com/documents/data-sheet/1N4148_1N4448.pdf" H 1700 6150 50  0001 C CNN
-F 4 "C81598" H 1700 6150 50  0001 C CNN "LCSC"
+F 4 "C2128" H 1700 6150 50  0001 C CNN "LCSC"
 	1    1700 6150
 	-1   0    0    -1
@@
 F 2 "Diode_SMD:D_SOD-323F" H 1700 6625 50  0001 C CNN
 F 3 "https://assets.nexperia.com/documents/data-sheet/1N4148_1N4448.pdf" H 1700 6800 50  0001 C CNN
-F 4 "C81598" H 1700 6800 50  0001 C CNN "LCSC"
+F 4 "C2128" H 1700 6800 50  0001 C CNN "LCSC"
 	1    1700 6800
 	-1   0    0    -1
@@
 F 2 "Diode_SMD:D_SOD-323F" H 2500 4575 50  0001 C CNN
 F 3 "https://assets.nexperia.com/documents/data-sheet/1N4148_1N4448.pdf" H 2500 4750 50  0001 C CNN
-F 4 "C81598" H 2500 4750 50  0001 C CNN "LCSC"
+F 4 "C2128" H 2500 4750 50  0001 C CNN "LCSC"
 	1    2500 4750
 	-1   0    0    -1
@@
 F 2 "Diode_SMD:D_SOD-323F" H 2500 5275 50  0001 C CNN
 F 3 "https://assets.nexperia.com/documents/data-sheet/1N4148_1N4448.pdf" H 2500 5450 50  0001 C CNN
-F 4 "C81598" H 2500 5450 50  0001 C CNN "LCSC"
+F 4 "C2128" H 2500 5450 50  0001 C CNN "LCSC"
 	1    2500 5450
 	-1   0    0    -1
@@
 F 2 "Diode_SMD:D_SOD-323F" H 2500 5975 50  0001 C CNN
 F 3 "https://assets.nexperia.com/documents/data-sheet/1N4148_1N4448.pdf" H 2500 6150 50  0001 C CNN
-F 4 "C81598" H 2500 6150 50  0001 C CNN "LCSC"
+F 4 "C2128" H 2500 6150 50  0001 C CNN "LCSC"
 	1    2500 6150
 	-1   0    0    -1
@@
 F 2 "Diode_SMD:D_SOD-323F" H 2500 6625 50  0001 C CNN
 F 3 "https://assets.nexperia.com/documents/data-sheet/1N4148_1N4448.pdf" H 2500 6800 50  0001 C CNN
-F 4 "C81598" H 2500 6800 50  0001 C CNN "LCSC"
+F 4 "C2128" H 2500 6800 50  0001 C CNN "LCSC"
 	1    2500 6800
 	-1   0    0    -1
@@
 F 2 "Diode_SMD:D_SOD-323F" H 3300 4575 50  0001 C CNN
 F 3 "https://assets.nexperia.com/documents/data-sheet/1N4148_1N4448.pdf" H 3300 4750 50  0001 C CNN
-F 4 "C81598" H 3300 4750 50  0001 C CNN "LCSC"
+F 4 "C2128" H 3300 4750 50  0001 C CNN "LCSC"
 	1    3300 4750
 	-1   0    0    -1
@@
 F 2 "Diode_SMD:D_SOD-323F" H 3300 5275 50  0001 C CNN
 F 3 "https://assets.nexperia.com/documents/data-sheet/1N4148_1N4448.pdf" H 3300 5450 50  0001 C CNN
-F 4 "C81598" H 3300 5450 50  0001 C CNN "LCSC"
+F 4 "C2128" H 3300 5450 50  0001 C CNN "LCSC"
 	1    3300 5450
 	-1   0    0    -1
@@
 F 2 "Diode_SMD:D_SOD-323F" H 3300 5975 50  0001 C CNN
 F 3 "https://assets.nexperia.com/documents/data-sheet/1N4148_1N4448.pdf" H 3300 6150 50  0001 C CNN
-F 4 "C81598" H 3300 6150 50  0001 C CNN "LCSC"
+F 4 "C2128" H 3300 6150 50  0001 C CNN "LCSC"
 	1    3300 6150
 	-1   0    0    -1
@@
 F 2 "Diode_SMD:D_SOD-323F" H 3300 6625 50  0001 C CNN
 F 3 "https://assets.nexperia.com/documents/data-sheet/1N4148_1N4448.pdf" H 3300 6800 50  0001 C CNN
-F 4 "C81598" H 3300 6800 50  0001 C CNN "LCSC"
+F 4 "C2128" H 3300 6800 50  0001 C CNN "LCSC"
 	1    3300 6800
 	-1   0    0    -1
@@
 F 2 "Diode_SMD:D_SOD-323F" H 3300 7325 50  0001 C CNN
 F 3 "https://assets.nexperia.com/documents/data-sheet/1N4148_1N4448.pdf" H 3300 7500 50  0001 C CNN
-F 4 "C81598" H 3300 7500 50  0001 C CNN "LCSC"
+F 4 "C2128" H 3300 7500 50  0001 C CNN "LCSC"
 	1    3300 7500
 	-1   0    0    -1
@@
 F 2 "Diode_SMD:D_SOD-323F" H 4100 4575 50  0001 C CNN
 F 3 "https://assets.nexperia.com/documents/data-sheet/1N4148_1N4448.pdf" H 4100 4750 50  0001 C CNN
-F 4 "C81598" H 4100 4750 50  0001 C CNN "LCSC"
+F 4 "C2128" H 4100 4750 50  0001 C CNN "LCSC"
 	1    4100 4750
 	-1   0    0    -1
@@
 F 2 "Diode_SMD:D_SOD-323F" H 4100 5275 50  0001 C CNN
 F 3 "https://assets.nexperia.com/documents/data-sheet/1N4148_1N4448.pdf" H 4100 5450 50  0001 C CNN
-F 4 "C81598" H 4100 5450 50  0001 C CNN "LCSC"
+F 4 "C2128" H 4100 5450 50  0001 C CNN "LCSC"
 	1    4100 5450
 	-1   0    0    -1
@@
 F 2 "Diode_SMD:D_SOD-323F" H 4100 6625 50  0001 C CNN
 F 3 "https://assets.nexperia.com/documents/data-sheet/1N4148_1N4448.pdf" H 4100 6800 50  0001 C CNN
-F 4 "C81598" H 4100 6800 50  0001 C CNN "LCSC"
+F 4 "C2128" H 4100 6800 50  0001 C CNN "LCSC"
 	1    4100 6800
 	-1   0    0    -1
@@
 F 2 "Diode_SMD:D_SOD-323F" H 4100 3925 50  0001 C CNN
 F 3 "https://assets.nexperia.com/documents/data-sheet/1N4148_1N4448.pdf" H 4100 4100 50  0001 C CNN
-F 4 "C81598" H 4100 4100 50  0001 C CNN "LCSC"
+F 4 "C2128" H 4100 4100 50  0001 C CNN "LCSC"
 	1    4100 4100
 	-1   0    0    -1
@@
 F 2 "Diode_SMD:D_SOD-323F" H 2500 3925 50  0001 C CNN
 F 3 "https://assets.nexperia.com/documents/data-sheet/1N4148_1N4448.pdf" H 2500 4100 50  0001 C CNN
-F 4 "C81598" H 2500 4100 50  0001 C CNN "LCSC"
+F 4 "C2128" H 2500 4100 50  0001 C CNN "LCSC"
 	1    2500 4100
 	-1   0    0    -1
@@
 F 2 "Diode_SMD:D_SOD-323F" H 1700 3925 50  0001 C CNN
 F 3 "https://assets.nexperia.com/documents/data-sheet/1N4148_1N4448.pdf" H 1700 4100 50  0001 C CNN
-F 4 "C81598" H 1700 4100 50  0001 C CNN "LCSC"
+F 4 "C2128" H 1700 4100 50  0001 C CNN "LCSC"
 	1    1700 4100
 	-1   0    0    -1
@@
 F 2 "Diode_SMD:D_SOD-323F" H 1700 4575 50  0001 C CNN
 F 3 "https://assets.nexperia.com/documents/data-sheet/1N4148_1N4448.pdf" H 1700 4750 50  0001 C CNN
-F 4 "C81598" H 1700 4750 50  0001 C CNN "LCSC"
+F 4 "C2128" H 1700 4750 50  0001 C CNN "LCSC"
 	1    1700 4750
 	-1   0    0    -1
@@
 F 2 "Diode_SMD:D_SOD-323F" H 1700 5275 50  0001 C CNN
 F 3 "https://assets.nexperia.com/documents/data-sheet/1N4148_1N4448.pdf" H 1700 5450 50  0001 C CNN
-F 4 "C81598" H 1700 5450 50  0001 C CNN "LCSC"
+F 4 "C2128" H 1700 5450 50  0001 C CNN "LCSC"
 	1    1700 5450
 	-1   0    0    -1
@@
 F 2 "Diode_SMD:D_SOD-323F" H 1700 7325 50  0001 C CNN
 F 3 "https://assets.nexperia.com/documents/data-sheet/1N4148_1N4448.pdf" H 1700 7500 50  0001 C CNN
-F 4 "C81598" H 1700 7500 50  0001 C CNN "LCSC"
+F 4 "C2128" H 1700 7500 50  0001 C CNN "LCSC"
 	1    1700 7500
 	-1   0    0    -1
@@
 F 2 "Diode_SMD:D_SOD-323F" H 3300 3925 50  0001 C CNN
 F 3 "https://assets.nexperia.com/documents/data-sheet/1N4148_1N4448.pdf" H 3300 4100 50  0001 C CNN
-F 4 "C81598" H 3300 4100 50  0001 C CNN "LCSC"
+F 4 "C2128" H 3300 4100 50  0001 C CNN "LCSC"
 	1    3300 4100
 	-1   0    0    -1

Commit message: Fixed header footprint
Parts:
- J1: footprint Connector_PinHeader_1.27mm:PinHeader_1x03_P1.27mm_Horizontal -> Connector_PinHeader_2.54mm:PinHeader_1x03_P2.54mm_Horizontal
Changed lines of the file:
@@
 F 0 "J1" H 8622 5774 50  0000 R CNN
 F 1 "SWD" H 8622 5683 50  0000 R CNN
-F 2 "Connector_PinHeader_1.27mm:PinHeader_1x03_P1.27mm_Horizontal" H 8650 5750 50  0001 C CNN
+F 2 "Connector_PinHeader_2.54mm:PinHeader_1x03_P2.54mm_Horizontal" H 8650 5750 50  0001 C CNN
 F 3 "~" H 8650 5750 50  0001 C CNN
 	1    8650 5750

Commit message: some changes; added license
Parts:
- removed C1, C10, C2, C3, C4, C6, C7: 100nf, Capacitor_SMD:C_0402_1005Metric, symbol Device:C_Small
- removed C11, C12, C5: 1uf, Capacitor_SMD:C_0402_1005Metric, symbol Device:C_Small
- removed C8, C9: 20pf, Capacitor_SMD:C_0402_1005Metric, symbol Device:C_Small
- removed D_0, D_1, D_2, D_3, D_4, D_5, D_6, D_7, D_8, D_9, D_BKSP1, D_DOT1, D_ENTER1, D_ESC1, D_FN1, D_MINUS1, D_NUMLK1, D_PLUS1, D_SLASH1, D_STAR1, D_TAB1: 1N4148, Diode_SMD:D_SOD-323F, symbol Diode:1N4148
- removed J1: SWD, Connector_PinHeader_2.54mm:PinHeader_1x03_P2.54mm_Horizontal, symbol Connector:Conn_01x03_Male
- removed J2: USB_C_Receptacle_USB2.0, Connector_USB:USB_C_Receptacle_GCT_USB4085, symbol Connector:USB_C_Receptacle_USB2.0
- removed R1: 10k, Resistor_SMD:R_0402_1005Metric, symbol Device:R_Small_US
- removed R2, R3: 5.1K, Resistor_SMD:R_0402_1005Metric, symbol Device:R_Small_US
- removed R4: 1.5K, Resistor_SMD:R_0402_1005Metric, symbol Device:R_Small_US
- removed SW_0, SW_ENTER1, SW_PLUS1: SW_Push, Keebio-Parts:MX-Alps-Choc-2U, symbol Switch:SW_Push
- removed SW_1, SW_2, SW_3, SW_4, SW_5, SW_6, SW_7, SW_8, SW_9, SW_BKSP1, SW_DOT1, SW_ESC1, SW_FN1, SW_MINUS1, SW_NUMLK1, SW_SLASH1, SW_STAR1, SW_TAB1: SW_Push, Keebio-Parts:MX-Alps-Choc-1U, symbol Switch:SW_Push
- removed U1: SRV05-4, Package_TO_SOT_SMD:SOT-23-6, symbol Power_Protection:SRV05-4
- removed U2: STM32F103C8Tx, Package_QFP:LQFP-48_7x7mm_P0.5mm, symbol MCU_ST_STM32F1:STM32F103C8Tx
- removed U3: XC6206PxxxMR, Package_TO_SOT_SMD:SOT-23, symbol Regulator_Linear:XC6206PxxxMR
- removed Y1: 8MHz, Crystal:Crystal_SMD_5032-2Pin_5.0x3.2mm, symbol Device:Crystal_Small
- added D_0, D_1, D_2, D_3, D_4, D_5, D_6, D_7, D_8, D_9, D_BKSP1, D_DOT1, D_ENTER1, D_ESC1, D_FN1, D_MINUS1, D_NUMLK1, D_PLUS1, D_SLASH1, D_STAR1, D_TAB1: 1N4148WS, Diode_SMD:D_SOD-323, symbol Diode:1N4148WS
- added D_LNM1, D_LPW1: LED, symbol Device:LED
- added R5, R6: 51R, symbol Device:R_Small_US
- added SW_0, SW_ENTER1, SW_PLUS1: MX-LED, Keebio-Parts:MX-Alps-Choc-2U, symbol MX_Alps_Hybrid:MX-LED
- added SW_1, SW_2, SW_3, SW_4, SW_5, SW_6, SW_7, SW_8, SW_9, SW_BKSP1, SW_DOT1, SW_ESC1, SW_FN1, SW_MINUS1, SW_NUMLK1, SW_SLASH1, SW_STAR1, SW_TAB1: MX-LED, Keebio-Parts:MX-Alps-Choc-1U, symbol MX_Alps_Hybrid:MX-LED
Connections:
- net labels added: LED_NUMLK, LED_POWER, LED_PWR
- net labels removed: +3.3V, +5V, BOOT0, CC1, CC2, DA+, DA-, DB+, DB-, NRST, PD0, PD1, SWDCLK, SWDIO, VBAT, VDD1, VDD2, VDD3, VDDA
- wire segments 112 -> 225
- no-connect marks 18 -> 0
Other:
- note added: "Indicator LEDs"
- note removed: "CC Pull-down"
- note removed: "Data Lines"
- note removed: "Debug Port"
- note removed: "Decoupling Capacitors"
- note removed: "ESD Protection"
- note removed: "MCU"
- note removed: "Oscillator"
- note removed: "Power Regulator"
- note removed: "Support Circuitry"
- note removed: "USB Port"

Commit message: v0.9pre
Parts:
- removed D_0, D_1, D_2, D_3, D_4, D_5, D_6, D_7, D_8, D_9, D_BKSP1, D_DOT1, D_ENTER1, D_ESC1, D_FN1, D_MINUS1, D_NUMLK1, D_PLUS1, D_SLASH1, D_STAR1, D_TAB1: 1N4148WS, Diode_SMD:D_SOD-323, symbol Diode:1N4148WS
- removed D_LNM1, D_LPW1: LED, symbol Device:LED
- removed R5, R6: 51R, symbol Device:R_Small_US
- added D1, D2, D3, D4, D5, D6: WS2813, LED_SMD:LED_WS2812_PLCC6_5.0x5.0mm_P1.6mm, symbol LED:WS2813
- added D10, D11, D12, D13, D14, D15, D16, D17, D7, D8, D9: BAT54C, Package_TO_SOT_SMD:SOT-23, symbol Diode:BAT54C
- added Q1: AO3401A, Package_TO_SOT_SMD:SOT-23, symbol Transistor_FET:AO3401A
- added R1: 10K, Resistor_SMD:R_0402_1005Metric, symbol Device:R_Small_US
- added R2: 150R, Resistor_SMD:R_0402_1005Metric, symbol Device:R_Small_US
- SW_0, SW_ENTER1, SW_PLUS1: footprint Keebio-Parts:MX-Alps-Choc-2U -> Keebio-Parts:MX-Alps-Choc-2U-StabFlip
Connections:
- net GND: now also D1.5 (GND), D1.6 (BIN), D2.5 (GND), D3.5 (GND), D4.5 (GND), D5.5 (GND), D6.5 (GND)
- net row1: now also D13.3, D7.3
- net row2: now also D14.3, D8.3
- net row3: now also D15.3, D9.3
- net row4: now also D10.3, D16.3
- net row5: now also D11.3, D17.3
- net row6: now also D12.3
- net at SW_ESC1.2 (ROW): now also D7.1
- net at SW_TAB1.2 (ROW): now also D7.2
- net at SW_FN1.2 (ROW): now also D13.1
- net at SW_BKSP1.2 (ROW): now also D13.2
- net at SW_NUMLK1.2 (ROW): now also D8.1
- net at SW_SLASH1.2 (ROW): now also D8.2
- net at SW_STAR1.2 (ROW): now also D14.1
- net at SW_MINUS1.2 (ROW): now also D14.2
- net at SW_7.2 (ROW): now also D9.1
- net at SW_8.2 (ROW): now also D9.2
- net at SW_9.2 (ROW): now also D15.1
- net at SW_PLUS1.2 (ROW): now also D15.2
- net at SW_4.2 (ROW): now also D10.1
- net at SW_5.2 (ROW): now also D10.2
- net at SW_6.2 (ROW): now also D16.1
- net at SW_1.2 (ROW): now also D11.1
- net at SW_2.2 (ROW): now also D11.2
- net at SW_3.2 (ROW): now also D17.1
- net at SW_ENTER1.2 (ROW): now also D17.2
- net at SW_0.2 (ROW): now also D12.1
- net at SW_DOT1.2 (ROW): now also D12.2
- net LED_PWR renamed LED_MATRIX
- net LED_MATRIX: now also Q1.2 (S)
- new net: Q1.1 (G), R2.1
- new net: D1.3 (DOUT), D3.4 (DIN), D5.6 (BIN)
- new net: D2.6 (BIN), D3.3 (DOUT), D5.4 (DIN)
- new net: D2.4 (DIN), D4.6 (BIN), D5.3 (DOUT)
- new net: D2.3 (DOUT), D4.4 (DIN), D6.6 (BIN)
- new net: D4.3 (DOUT), D6.4 (DIN)
- new net +5V: D1.2 (VDD), D2.2 (VDD), D3.2 (VDD), D4.2 (VDD), D5.2 (VDD), D6.2 (VDD), Q1.3 (D), R1.1
- new net BL_CONTROL: D1.4 (DIN), D3.6 (BIN)
- new net LED_CONTROL: R1.2, R2.2
- no-connect marks 0 -> 8
Other:
- note removed: "Indicator LEDs"
- moved on the sheet: SW_0, SW_1, SW_2, SW_3, SW_4, SW_5, SW_6, SW_7, SW_8, SW_9, SW_BKSP1, SW_DOT1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
