File: Numpad.kicad_pcb (KiCad board)
At the start: 2 copper layers, 94 x 162.6 mm, 48 parts, among them SW1 SW_Push, SW10 SW_Push, SW11 SW_Push, SW12 SW_Push, SW13 SW_Push, SW14 SW_Push, SW15 SW_Push, SW16 SW_Push, SW17 SW_Push, SW18 SW_Push, SW19 SW_Push, SW2 SW_Push, SW20 SW_Push, SW21 SW_Push, SW22 SW_Push, SW3 SW_Push, SW4 SW_Push, SW5 SW_Push, SW6 SW_Push, SW7 SW_Push, SW8 SW_Push, SW9 SW_Push, U1 ProMicro

Commit message: changed schematic to use labels
Connections:
- net Net-(D1-Pad1) renamed col1
- net Net-(D10-Pad1) renamed col2
- net Net-(D12-Pad1) renamed col3
- net Net-(D18-Pad1) renamed col4
- net Net-(SW10-Pad2) renamed row3
- net Net-(SW11-Pad2) renamed row4
- net Net-(SW12-Pad2) renamed row5
- net Net-(SW13-Pad2) renamed row1
- net Net-(SW14-Pad2) renamed row2
- net Net-(SW18-Pad2) renamed row6

Commit message: Finished
Parts:
- removed HOLE1, HOLE2, HOLE3, HOLE4: MountingHole_3.2mm_M3, MountingHole:MountingHole_3.2mm_M3
- removed the SW1 at (66.0, 35.6)
- added C1: 100nf, Capacitor_SMD:C_0402_1005Metric, F.Cu at (38.1, 34.9)
- added C10: 100nf, Capacitor_SMD:C_0402_1005Metric, F.Cu at (36.8, 38.7)
- added C11: 1uf, Capacitor_SMD:C_0402_1005Metric, F.Cu at (57.1, 27.9)
- added C12: 1uf, Capacitor_SMD:C_0402_1005Metric, F.Cu at (54.6, 30.5)
- added C2: 100nf, Capacitor_SMD:C_0402_1005Metric, F.Cu at (48.3, 45.1)
- added C3: 100nf, Capacitor_SMD:C_0402_1005Metric, F.Cu at (50.8, 35.6)
- added C4: 100nf, Capacitor_SMD:C_0402_1005Metric, F.Cu at (41.9, 32.4)
- added C5: 1uf, Capacitor_SMD:C_0402_1005Metric, F.Cu at (37.5, 40.6)
- added C6: 100nf, Capacitor_SMD:C_0402_1005Metric, F.Cu at (36.2, 40.6)
- added C7: 100nf, Capacitor_SMD:C_0402_1005Metric, F.Cu at (55.2, 33.0)
- added C8: 20pf, Capacitor_SMD:C_0402_1005Metric, F.Cu at (27.9, 33.7)
- added C9: 20pf, Capacitor_SMD:C_0402_1005Metric, F.Cu at (27.9, 36.2)
- added H1: MountingHole_Pad, MountingHole:MountingHole_3.2mm_M3_Pad, F.Cu at (21.6, 21.6)
- added H2: MountingHole_Pad, MountingHole:MountingHole_3.2mm_M3_Pad, F.Cu at (105.4, 21.6)
- added H3: MountingHole_Pad, MountingHole:MountingHole_3.2mm_M3_Pad, F.Cu at (21.6, 174.0)
- added H4: MountingHole_Pad, MountingHole:MountingHole_3.2mm_M3_Pad, F.Cu at (105.4, 174.0)
- added J1: SWD, Connector_PinHeader_1.27mm:PinHeader_1x03_P1.27mm_Horizontal, F.Cu at (47.6, 30.5)
- added J2: USB4085-GF-A_REVA, USB4085:GCT_USB4085-GF-A_REVA, F.Cu at (63.5, 19.1)
- added R1: 10k, Resistor_SMD:R_0402_1005Metric, F.Cu at (44.5, 31.1)
- added R2: 5.1K, Resistor_SMD:R_0402_1005Metric, F.Cu at (72.4, 21.6)
- added R3: 5.1K, Resistor_SMD:R_0402_1005Metric, F.Cu at (55.9, 21.6)
- added U2: STM32F103C8Tx, Package_QFP:LQFP-48_7x7mm_P0.5mm, F.Cu at (44.5, 38.7)
- added U3: XC6206PxxxMR, Package_TO_SOT_SMD:SOT-23, F.Cu at (57.1, 30.5)
- added Y1: 8MHz, Crystal:Crystal_SMD_5032-2Pin_5.0x3.2mm, F.Cu at (33.0, 34.9)
- D1, D10, D11, D12, D13, D14, D15, D16, D17, D18, D19, D2, D20, D21, D3, D4, D5, D6, D7, D8, D9: footprint Diode_THT:D_DO-35_SOD27_P7.62mm_Horizontal -> Diode_SMD:D_SOD-123; moved to F.Cu
- U1: value ProMicro -> SRV05-4; footprint ProMicro:ProMicro -> Package_TO_SOT_SMD:SOT-23-6
- moved U1 25.9 mm to (66.0, 29.2), turned to 180 degrees
- moved D10 6.98 mm to (63.5, 116.8)
- moved D15 6.98 mm to (82.5, 116.8)
- moved D3 6.98 mm to (44.5, 97.8)
- moved D4 6.98 mm to (44.5, 116.8)
- moved D9 6.98 mm to (63.5, 97.8)
- moved D11 6.98 mm to (63.5, 135.9)
- moved D17 6.98 mm to (82.5, 154.9)
- moved D5 6.98 mm to (44.5, 135.9)
- moved D13 6.35 mm to (82.5, 78.1)
- moved D19 6.35 mm to (101.6, 78.1)
- moved D2 6.35 mm to (44.5, 78.1)
- moved D8 6.35 mm to (63.5, 78.1)
- moved D12 6.35 mm to (82.5, 52.7)
- moved D18 6.35 mm to (101.6, 52.7)
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- renumbered SW2 to SW1, SW11 to SW10, SW12 to SW11, SW13 to SW12, SW14 to SW13, SW15 to SW14, SW16 to SW15, SW17 to SW16, SW18 to SW17, SW19 to SW18, SW20 to SW19, SW3 to SW2, SW21 to SW20, SW22 to SW21, SW4 to SW3, SW5 to SW4, SW6 to SW5, SW7 to SW6, SW8 to SW7, SW9 to SW8, SW10 to SW9
Connections:
- U1 pad 2: Net-(U1-Pad2) -> GND
- U1 pad 4: Net-(U1-Pad4) -> DA+
- U1 pad 5: Net-(U1-Pad5) -> +5V
- U1 pad 6: Net-(U1-Pad6) -> DA-
Routing:
- net GND: track 0.00 -> 593.5 mm, vias 0 -> 2
- net VBAT: track 0.00 -> 47.9 mm, vias 0 -> 3
- net Net-(SW1-Pad2): track 42.4 -> 0.00 mm
- net Net-(SW1-Pad1): track 38.0 -> 0.00 mm
- net DA+: track 0.00 -> 31.3 mm, vias 0 -> 2
- net DA-: track 0.00 -> 30.9 mm
- net col1: track 144.0 -> 117.4 mm, vias 0 -> 2
- net +5V: track 0.00 -> 23.9 mm, vias 0 -> 2
- net col4: track 174.2 -> 157.4 mm, vias 0 -> 2
- net col2: track 122.6 -> 107.1 mm
- net Net-(C8-Pad1): track 0.00 -> 14.1 mm
- net Net-(C9-Pad1): track 0.00 -> 12.8 mm
- net Net-(J1-Pad3): track 0.00 -> 9.72 mm, vias 0 -> 2
- net /CC1: track 0.00 -> 9.01 mm
- net col3: track 163.4 -> 156.0 mm, vias 0 -> 2
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- added copper zone on B.Cu, net GND
Other:
- net class Default: clearance 0.2 -> 0.127; trace_width 0.25 -> 0.127; via_dia 0.8 -> 0.6; via_drill 0.4 -> 0.3
- rule trace_clearance: 0.2 -> 0.127
- board text added: "NumpadA v0.2 Standalone by Dmitry Kudriavtsev"
- board text removed: "NumpadA v0.1 by Dmitry Kudriavtsev"
- board text removed: "Reset"

Commit message: ground plane
Connections:
- U2 pad 17: Net-(U2-Pad17) -> row6
- U2 pad 18: Net-(U2-Pad18) -> row5
- U2 pad 19: Net-(U2-Pad19) -> row4
- U2 pad 20: Net-(U2-Pad20) -> row3
- U2 pad 42: row6 -> Net-(U2-Pad42)
- U2 pad 43: row5 -> Net-(U2-Pad43)
- U2 pad 45: row4 -> Net-(U2-Pad45)
- U2 pad 46: row3 -> Net-(U2-Pad46)
Routing:
- net GND: track 593.5 -> 34.6 mm, vias 2 -> 8
- net VBAT: track 47.9 -> 62.5 mm
- net row6: track 185.9 -> 174.6 mm, vias 2 -> 0
- net col3: track 156.0 -> 145.1 mm
- net row5: track 186.5 -> 178.6 mm, vias 2 -> 0
- net row4: track 143.3 -> 136.1 mm, vias 2 -> 0
- net row3: track 146.4 -> 139.6 mm, vias 2 -> 0
- net col4: track 157.4 -> 155.7 mm, vias 2 -> 0
- net DA-: track 30.9 -> 32.5 mm
- net /CC1: track 9.01 -> 10.2 mm
- net +5V: track 23.9 -> 25.0 mm
- net Net-(J1-Pad3): track 9.72 -> 8.98 mm, vias 2 -> 0
- net Net-(R1-Pad1): track 3.97 -> 4.71 mm
- net Net-(C8-Pad1): track 14.1 -> 14.8 mm
- net col1: track 117.4 -> 117.7 mm, vias 2 -> 0
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
Commit message: D+ pullup and some other things
Parts:
- added R4: 1.5K, Resistor_SMD:R_0402_1005Metric, F.Cu at (61.0, 27.9)
Routing:
- net VBAT: track 62.5 -> 72.4 mm
- net GND: track 34.6 -> 38.5 mm
- net DA+: track 31.7 -> 32.8 mm

Commit message: finalized v0.2
Other:
- board text added: "NumpadA v0.2 Standalone by Inexpensive Computers"
- board text removed: "NumpadA v0.2 Standalone by Dmitry Kudriavtsev"
Changed lines of the file:
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@@
       (drillshape 0)
       (scaleselection 1)
-      (outputdirectory "/Users/dmitry/Documents/numpad-gerber/"))
+      (outputdirectory "./"))
   )
   (net 0 "")
@@
     (tags capacitor)
     (attr smd)
-    (fp_text reference C8 (at 0 -1.17) (layer F.SilkS)
+    (fp_text reference C8 (at 2.54 0) (layer F.SilkS)
       (effects (font (size 1 1) (thickness 0.15)))
     )
@@
     (tags capacitor)
     (attr smd)
-    (fp_text reference C9 (at 0 -1.17) (layer F.SilkS)
+    (fp_text reference C9 (at 2.54 0) (layer F.SilkS)
       (effects (font (size 1 1) (thickness 0.15)))
     )
@@
     (tags "mounting hole 3.2mm m3")
     (attr virtual)
-    (fp_text reference H1 (at 0 -4.2) (layer F.SilkS)
+    (fp_text reference H1 (at 0 -4.2) (layer F.SilkS) hide
       (effects (font (size 1 1) (thickness 0.15)))
     )
@@
     (tags "mounting hole 3.2mm m3")
     (attr virtual)
-    (fp_text reference H2 (at 0 -4.2) (layer F.SilkS)
+    (fp_text reference H2 (at 0 -4.2) (layer F.SilkS) hide
       (effects (font (size 1 1) (thickness 0.15)))
     )
@@
     (tags "mounting hole 3.2mm m3")
     (attr virtual)
-    (fp_text reference H3 (at 0 -4.2) (layer F.SilkS)
+    (fp_text reference H3 (at 0 -4.2) (layer F.SilkS) hide
       (effects (font (size 1 1) (thickness 0.15)))
     )
@@
     (tags "mounting hole 3.2mm m3")
     (attr virtual)
-    (fp_text reference H4 (at 0 -4.2) (layer F.SilkS)
+    (fp_text reference H4 (at 0 -4.2) (layer F.SilkS) hide
       (effects (font (size 1 1) (thickness 0.15)))
     )
@@
     (descr "Through hole angled pin header, 1x03, 1.27mm pitch, 4.0mm pin length, single row")
     (tags "Through hole angled pin header THT 1x03 1.27mm single row")
-    (fp_text reference J1 (at 2.4325 -1.635 90) (layer F.SilkS)
+    (fp_text reference J1 (at -1.905 1.27 180) (layer F.SilkS)
       (effects (font (size 1 1) (thickness 0.15)))
     )
@@
   (module USB4085:GCT_USB4085-GF-A_REVA (layer F.Cu)
     (at 63.5 19.05 180)
-    (fp_text reference J2 (at -6.35 -1.27 90) (layer F.SilkS)
-      (effects (font (size 1.00015 1.00015) (thickness 0.015)))
+    (fp_text reference J2 (at 0 -5.715 180) (layer F.SilkS)
+      (effects (font (size 1.00015 1.00015) (thickness 0.15)))
     )
     (fp_text value USB4085-GF-A_REVA (at 9.18404 5.83792) (layer F.Fab)
@@
     (tags SOT-23-6)
     (attr smd)
-    (fp_text reference U1 (at -2.54 0 270) (layer F.SilkS)
+    (fp_text reference U1 (at 0 2.54) (layer F.SilkS)
       (effects (font (size 1 1) (thickness 0.15)))
     )
@@
     )
   )
-  (gr_text "NumpadA v0.2 Standalone\nby Dmitry Kudriavtsev" (at 62.865 38.1) (layer F.SilkS)
+  (gr_text "NumpadA v0.2 Standalone\nby Inexpensive Computers" (at 62.23 41.91) (layer F.SilkS)
     (effects (font (size 2 2) (thickness 0.15)) (justify left))
   )
@@
   (segment (start 43.7 42.8975) (end 43.7 43.635) (width 0.127) (layer F.Cu) (net 33))
   (via (at 67.31 29.21) (size 0.6) (drill 0.3) (layers F.Cu B.Cu) (net 34))
-  (via (at 59.69 30.48) (size 0.6) (drill 0.3) (layers F.Cu B.Cu) (net 38))
-  (via (at 64.77 29.21) (size 0.6) (drill 0.3) (layers F.Cu B.Cu) (net 38))
   (via (at 27.305 34.925) (size 0.6) (drill 0.3) (layers F.Cu B.Cu) (net 34))
   (via (at 34.925 38.735) (size 0.6) (drill 0.3) (layers F.Cu B.Cu) (net 34))
@@
   (segment (start 37.86 38.985) (end 39.55 38.985) (width 0.127) (layer F.Cu) (net 37))
   (segment (start 37.315 38.735) (end 37.61 38.735) (width 0.127) (layer F.Cu) (net 37))
+  (via (at 59.69 30.48) (size 0.6) (drill 0.3) (layers F.Cu B.Cu) (net 38))
+  (via (at 64.77 29.21) (size 0.6) (drill 0.3) (layers F.Cu B.Cu) (net 38))
   (segment (start 63.5 30.48) (end 64.77 29.21) (width 0.127) (layer B.Cu) (net 38))
   (segment (start 61.375 22.184619) (end 61.375 23.075) (width 0.127) (layer F.Cu) (net 38))

Commit message: v0.3
Parts:
- moved C8 4.58 mm to (31.8, 36.2), turned to 270 degrees
- moved C9 4.58 mm to (31.8, 38.7), turned to 90 degrees
- moved Y1 2.84 mm to (34.3, 37.5)
- moved C6 2.72 mm to (38.0, 42.7), turned to 0 degrees
- moved C1 1.76 mm to (39.6, 34.0)
- moved R1 1.59 mm to (43.7, 32.5), turned to 90 degrees
- moved C10 1.42 mm to (37.5, 40.0), turned to 90 degrees
- moved R4 1.27 mm to (61.0, 29.2)
- moved C5 1.04 mm to (38.0, 41.5), turned to 0 degrees
- moved C2 0.79 mm to (48.3, 44.3), turned to 90 degrees
Routing:
- net col1: track 117.7 -> 124.7 mm, vias 0 -> 2
- net GND: track 38.5 -> 43.4 mm, vias 8 -> 7
- net +5V: track 25.3 -> 30.0 mm
- net Net-(C8-Pad1): track 14.8 -> 10.4 mm
- net Net-(R1-Pad1): track 4.71 -> 1.58 mm
- net Net-(C9-Pad1): track 12.8 -> 9.74 mm
- net DA-: track 32.5 -> 31.7 mm
- net col4: track 155.7 -> 156.5 mm, vias 0 -> 2
- net VBAT: track 72.4 -> 71.8 mm
- net col2: track 106.8 -> 106.6 mm, vias 2 -> 0
- net row1: vias 2 -> 0
Other:
- board text added: "NumpadA v0.3 Standalone by Inexpensive Computers"
- board text removed: "NumpadA v0.2 Standalone by Inexpensive Computers"

Commit message: v0.3 minor tweaks
Parts:
- moved C2 1.09 mm to (47.2, 44.7), turned to 0 degrees
- moved C7 0.63 mm to (54.6, 33.0)
Routing:
- net GND: track 43.4 -> 49.4 mm, vias 7 -> 6
- net VBAT: track 71.8 -> 75.9 mm
