File: mcu.sch (KiCad schematic (older format))
At the start: 24 parts

Commit message: v0.9pre
Parts:
- added F1: SMD0805P050TF, Fuse:Fuse_0805_2012Metric_Castellated, symbol Device:Polyfuse_Small
- added R3: 1M, Resistor_SMD:R_0402_1005Metric, symbol Device:R_Small_US
- J1: renamed from J?; footprint Connector_USB:USB_C_Receptacle_GCT_USB4085 -> Connector_USB:USB_C_Receptacle_HRO_TYPE-C-31-M-12
- gave numbers to parts that had none: 23
Connections:
- net +5V: now also F1.2; no longer J1.A4 (VBUS), J1.A9 (VBUS), J1.B4 (VBUS), J1.B9 (VBUS)
- net DA+: now also U3.4 (IO3)
- net DA-: now also U3.3 (IO2); no longer U3.4 (IO3)
- net GND: now also R3.2; no longer J1.S1 (SHIELD)
- net row1: now also U1.21 (PB10); no longer U1.46 (PB9)
- net row2: now also U1.20 (PB2); no longer U1.22 (PB11)
- net row3: now also U1.19 (PB1); no longer U1.21 (PB10)
- net row4: now also U1.18 (PB0); no longer U1.20 (PB2)
- net row5: now also U1.17 (PA7); no longer U1.19 (PB1)
- net row6: now also U1.16 (PA6); no longer U1.18 (PB0)
- net LED_NUMLK: now reaches U1.11 (PA1)
- net BL_CONTROL: now reaches U1.15 (PA5)
- net LED_CONTROL: now reaches U1.42 (PB6)
- new net: F1.1, J1.A4 (VBUS), J1.A9 (VBUS), J1.B4 (VBUS), J1.B9 (VBUS)
- new net: J1.S1 (SHIELD), R3.1
- no-connect marks 20 -> 19

Commit message: v0.9
Parts:
- F1: LCSC (none) -> C20978
- R26: renamed from R3; LCSC (none) -> C25082
- renumbered C7 to C1, C16 to C10, C18 to C11, C17 to C12, C10 to C2, C12 to C3, C13 to C4, C14 to C5, C8 to C6, C9 to C7, C11 to C8, C15 to C9, R12 to R25, R13 to R27, R11 to R28, R14 to R29, U2 to U1, U3 to U2, U1 to U3
Connections:
- net col3: now also U3.3 (PC14); no longer U3.13 (PA3)
- net col4: now also U3.2 (PC13); no longer U3.12 (PA2)
- net row1: now also U3.38 (PA15); no longer U3.21 (PB10)
- no-connect marks 19 -> 16
